File: pcb/fr99.kicad_sch (KiCad schematic)
At the start: 20 parts, among them M1 SD_Module, P1 CONN_02X18, SW2 SW_PUSH, U1 74HCT541, U2 74HCT541, U3 74HCT541, U4 74HCT377, U5 62256, U6 ATMEGA8515-P

Commit message: Cleanup footprints and library links
Parts:
- removed C7: 1nF, flashcart-footprints:C_C, symbol Device:C
- C1, C2, C3, C4, C5, C6: footprint flashcart-footprints:C_C -> fr99-footprints:C_C
- D1: footprint LEDs:LED-5MM -> LED_THT:LED_D5.0mm
- M1: footprint flashcart-footprints:SD_MODULE -> fr99-footprints:SD_MODULE; symbol SD_Module -> fr99-components:SD_Module
- P1: footprint flashcart-footprints:BUS_CART -> fr99-footprints:BUS_CART
- R1, R2, R3: footprint Resistors_ThroughHole:Resistor_Horizontal_RM10mm -> Resistor_THT:R_Axial_DIN0207_L6.3mm_D2.5mm_P10.16mm_Horizontal
- SW2: footprint Buttons_Switches_ThroughHole:SW_PUSH_SMALL -> Button_Switch_THT:SW_PUSH_6mm_H5mm
- U1, U2, U3, U4: footprint Housings_DIP:DIP-20_W7.62mm -> Package_DIP:DIP-20_W7.62mm
- U5: footprint Housings_DIP:DIP-28_W15.24mm -> Package_DIP:DIP-28_W15.24mm; symbol HM62256BLP-7 -> Memory_RAM:HM62256BLP
- U6: footprint Housings_DIP:DIP-40_W15.24mm -> Package_DIP:DIP-40_W15.24mm; symbol ATMEGA8515-P -> MCU_Microchip_ATmega:ATmega8515-16P
Connections:
- net +5V: now also M1.6 (5V), U5.28 (VCC), U6.40 (VCC)
- net A0: now also U5.10 (A0), U6.39 (PA0)
- net A1: now also U5.9 (A1), U6.38 (PA1)
- net A10: now also U5.21 (A10), U6.29 (PE2)
- net A11: now also U5.23 (A11), U6.25 (PC4)
- net A12: now also U5.2 (A12), U6.26 (PC5)
- net A13: now also U5.26 (A13), U6.27 (PC6)
- net A14: now also U5.1 (A14), U6.28 (PC7)
- net A2: now also U5.8 (A2), U6.37 (PA2)
- net A3: now also U5.7 (A3), U6.36 (PA3)
- net A4: now also U5.6 (A4), U6.35 (PA4)
- net A5: now also U5.5 (A5), U6.34 (PA5)
- net A6: now also U5.4 (A6), U6.33 (PA6)
- net A7: now also U5.3 (A7), U6.32 (PA7)
- net A8: now also U5.25 (A8), U6.31 (PE0)
- net A9: now also U5.24 (A9), U6.30 (PE1)
- net BUSE: now also U6.24 (PC3)
- net D0: now also U5.11 (Q0), U6.10 (PD0)
- net D1: now also U5.12 (Q1), U6.11 (PD1)
- net D2: now also U5.13 (Q2), U6.12 (PD2)
- net D3: now also U5.15 (Q3), U6.13 (PD3)
- net D4: now also U5.16 (Q4), U6.14 (PD4)
- net D5: now also U5.17 (Q5), U6.15 (PD5)
- net D6: now also U5.18 (Q6), U6.16 (PD6)
- net D7: now also U5.19 (Q7), U6.17 (PD7)
- net GND: now also M1.1 (GND), M1.8 (GND), U5.14 (GND), U6.20 (GND)
- net at U4.12 (Q4): now also U6.7 (PB6)
- net at U4.15 (Q5): now also U6.6 (PB5)
- net at U1.18 (Y0): now also U5.22 (~{OE}), U6.22 (PC1)
- net at R3.2, SW2.2: now also U6.9 (~{RESET})
- net at R2.2: now also U6.8 (PB7)
- new net: U5.20 (~{CS}), U6.21 (PC0)
- new net: U5.27 (~{WE}), U6.23 (PC2)
- new net: M1.5 (CS), U6.1 (PB0)
- new net: M1.3 (SCK), U6.2 (PB1)
- new net: M1.4 (MOSI), U6.3 (PB2)
- new net: M1.2 (MISO), U6.4 (PB3)
Other:
- note removed: "1"
- moved on the sheet: C1, C2, C3, C4, C5, C6
